File: IF-GBP-02.kicad_sch (KiCad schematic)
At the start: 82 parts, among them CN1 Print Motor, CN2 GB Printer Print Head, CN3 Gameboy Link Port, IC1 4A 8D1 - BGA6489, IC2 TMP87CM40AF, IC3 LH5164, IC5 TD62593A, IC6 TD62593A, IC7 458F - FMMT458TA SOT23-5, J2 Battery Connectors, Q1 B1326, Q10 BR - BCW60DR, Q11 BR - BCW60DR, Q14 24 - DTC114ECA, Q2 FR - 2SA1037, Q3 BR - BCW60DR, Q4 FR - 2SA1037, Q5 24 - DTC114ECA, Q6 BF RD - RT9169, Q7 CF RD - 2SC3650, Q8 BR - BCW60DR, Q9 FR - 2SA1037, SW1 SW_MEC_5E, SW2 SW_DPDT_x2, X1 8 MHz

Commit message: Add files via upload
Parts:
- removed Q6: BF RD - RT9169, Gameboy Printer:SOT89 Transistor, symbol Regulator_Linear:HT75xx-1-SOT89
- added Q6: BF RD, Gameboy Printer:SOT89 Transistor, symbol Device:Q_PNP_BEC
- IC7: value 458F - FMMT458TA SOT23-5 -> 458F
- Q4, Q9: value FR - 2SA1037 -> FR
- Q7: value CF RD - 2SC3650 -> CF RD
- Q8: value BR - BCW60DR -> BR
Connections:
- net 9V.Postfuse is gone; now on net GND: C1.1, F2.1, Q1.3 (E), R1.1, R16.2, R17.2, R21.1
- net Resistor.Bus is gone; now on net VCC: NR1.5 (R4.2), NR1.6 (R3.2), NR1.7 (R2.2), NR1.8 (R1.2), NR2.5 (R4.2), NR2.6 (R3.2), NR2.7 (R2.2), NR2.8 (R1.2), NR3.5 (R4.2), NR3.6 (R3.2), NR3.7 (R2.2), NR3.8 (R1.2), NR4.4 (R4.1), NR4.6 (R3.2), NR4.7 (R2.2), NR4.8 (R1.2)
- net Route10 is gone; now on net GND: C2.2, IC1.2 (GND), R9.1
- net Route17 is gone; now on net GND: C3.2, C5.1, Q2.3 (C)
- net Route22 is gone; now on net GND: C18.1, IC7.3 (C), R22.2
- net Route26 is gone; now on an unnamed net: C6.2, Q14.3 (C), R14.2
- net Route28 is gone; now on net GND: C12.2, Q10.2 (E)
- net CN1.P2: now also Q6.2 (E)
- net VCC: now also Q6.3 (C)
- net 9V.F1: no longer names the net of F1.2, SW2.5 (B)
- net 9V.Prefuse: no longer names the net of F2.2, R26.2, SW2.6 (C)
- net LED.Anode: no longer names the net of C2.1, C4.2, CN2.1 (Pin_1), CN2.2 (Pin_2), L1.1, L2.1, LED1.2 (A)
- net LED.Cathode: no longer names the net of LED1.1 (K), R23.2
- net Route1: no longer names the net of D1.2 (A), L1.2, Q1.2 (C)
- net Route12: no longer names the net of Q7.1 (B), Q9.3 (C)
- net Route13: no longer names the net of Q8.1 (B), Q9.1 (B), R34.2
- net Route14: no longer names the net of Q8.2 (E), Q9.2 (E), R35.1, R36.2
- net Route15: no longer names the net of IC1.3 (+), Q11.2 (E), R8.2
- net Route16: no longer names the net of Q8.3 (C)
- net Route16: now also Q6.1 (B)
- net Route19: no longer names the net of C6.1, D5.1 (K), Q11.1 (B), Q4.2 (E), R14.1, R16.1
- net Route2: no longer names the net of Q1.1 (B), R1.2, R2.2
- net Route20: no longer names the net of IC7.1 (E), Q3.1 (B), R7.2, R8.1
- net Route21: no longer names the net of C18.2, IC7.2 (B), R21.2, R22.1
- net Route23: no longer names the net of Q4.1 (B), Q5.3 (C)
- net Route24: no longer names the net of Q4.3 (C), Q5.1 (B)
- net Route25: no longer names the net of Q11.3 (C), R17.1
- net Route27: no longer names the net of Q10.1 (B), R32.1
- net Route3: no longer names the net of R2.1, R3.1
- net Route4: no longer names the net of R3.2, R4.1
- net Route5: no longer names the net of R4.2, R5.2
- net Route6: no longer names the net of Q2.2 (E), R5.1
- net Route7: no longer names the net of Q2.1 (B), Q3.3 (C)
- net Route8: no longer names the net of IC1.1, R10.1, R12.2, R9.2
- net Route9: no longer names the net of C4.1, R12.1
Other:
- moved on the sheet: C1, C12, C14, C15, C16, C17, C18, C19, C2, C20, C3, C4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

Commit message: Add files via upload
Parts:
- removed IC1: 4A 8D1 - BGA6489, Gameboy Printer:SOT89 Transistor, symbol Amplifier_Operational:TL064
- added IC1: 4A 8D1, Gameboy Printer:SOT89 Transistor, symbol Device:Q_PNP_BCE
Connections:
- net GND: now also IC1.2 (C)
- net at R10.1, R12.2, R9.2: now also IC1.1 (B)
- net at Q11.2 (E), R8.2: now also IC1.3 (E)
Changed lines of the file:
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@@
   (junction (at 501.65 251.46) (diameter 0) (color 0 0 0 0)
   )
+  (junction (at 363.22 242.57) (diameter 0) (color 0 0 0 0)
+  )
   (junction (at 501.65 262.89) (diameter 0) (color 0 0 0 0)
   )
@@
   )
   (junction (at 424.18 281.94) (diameter 0) (color 0 0 0 0)
-  )
-  (junction (at 367.03 242.57) (diameter 0) (color 0 0 0 0)
   )
   (junction (at 397.51 123.19) (diameter 0) (color 0 0 0 0)
@@
     (stroke (width 0) (type default) (color 0 0 0 0))
   )
-  (wire (pts (xy 367.03 231.14) (xy 363.22 231.14))
-    (stroke (width 0) (type default) (color 0 0 0 0))
-  )
   (wire (pts (xy 387.35 151.13) (xy 396.24 151.13))
     (stroke (width 0) (type default) (color 0 0 0 0))
@@
     (stroke (width 0) (type default) (color 0 0 0 0))
   )
+  (wire (pts (xy 363.22 242.57) (xy 326.39 242.57))
+    (stroke (width 0) (type default) (color 0 0 0 0))
+  )
   (wire (pts (xy 382.27 123.19) (xy 397.51 123.19))
     (stroke (width 0) (type default) (color 0 0 0 0))
@@
     (stroke (width 0) (type default) (color 0 0 0 0))
   )
-  (wire (pts (xy 424.18 229.87) (xy 424.18 267.97))
+  (wire (pts (xy 424.18 234.95) (xy 424.18 267.97))
     (stroke (width 0) (type default) (color 0 0 0 0))
   )
@@
     (stroke (width 0) (type default) (color 0 0 0 0))
   )
-  (wire (pts (xy 367.03 242.57) (xy 367.03 231.14))
+  (wire (pts (xy 363.22 242.57) (xy 363.22 231.14))
     (stroke (width 0) (type default) (color 0 0 0 0))
   )
@@
     (stroke (width 0) (type default) (color 0 0 0 0))
   )
-  (wire (pts (xy 370.84 226.06) (xy 370.84 250.19))
+  (wire (pts (xy 374.65 226.06) (xy 374.65 250.19))
     (stroke (width 0) (type default) (color 0 0 0 0))
   )
@@
     (stroke (width 0) (type default) (color 0 0 0 0))
   )
-  (wire (pts (xy 367.03 242.57) (xy 326.39 242.57))
-    (stroke (width 0) (type default) (color 0 0 0 0))
-  )
   (wire (pts (xy 396.24 180.34) (xy 396.24 167.64))
     (stroke (width 0) (type default) (color 0 0 0 0))
   )
-  (wire (pts (xy 367.03 255.27) (xy 367.03 242.57))
+  (wire (pts (xy 363.22 255.27) (xy 363.22 242.57))
     (stroke (width 0) (type default) (color 0 0 0 0))
   )
@@
     (stroke (width 0) (type default) (color 0 0 0 0))
   )
-  (wire (pts (xy 452.12 229.87) (xy 424.18 229.87))
+  (wire (pts (xy 424.18 234.95) (xy 459.74 234.95))
     (stroke (width 0) (type default) (color 0 0 0 0))
   )
@@
     (stroke (width 0) (type default) (color 0 0 0 0))
   )
+  (wire (pts (xy 374.65 226.06) (xy 370.84 226.06))
+    (stroke (width 0) (type default) (color 0 0 0 0))
+  )
   (wire (pts (xy 436.88 328.93) (xy 436.88 339.09))
     (stroke (width 0) (type default) (color 0 0 0 0))
@@
     (stroke (width 0) (type default) (color 0 0 0 0))
   )
-  (wire (pts (xy 370.84 250.19) (xy 374.65 250.19))
+  (wire (pts (xy 363.22 255.27) (xy 367.03 255.27))
     (stroke (width 0) (type default) (color 0 0 0 0))
   )
@@
     (effects (font (size 1.27 1.27)) (justify left bottom))
   )
+  (label "GND" (at 459.74 224.79 90)
+    (effects (font (size 1.27 1.27)) (justify left bottom))
+  )
   (label "D3" (at 190.5 96.52 270)
     (effects (font (size 1.27 1.27)) (justify right bottom))
@@
     (effects (font (size 1.27 1.27)) (justify right bottom))
   )
-  (label "GND" (at 459.74 224.79 90)
-    (effects (font (size 1.27 1.27)) (justify left bottom))
-  )
   (label "D6" (at 209.55 91.44 0)
     (effects (font (size 1.27 1.27)) (justify left bottom))
@@
     (pin "1")
     (pin "2")
+  )
+  (symbol (lib_id "Device:Q_PNP_BCE") (at 462.28 229.87 0) (mirror y) (unit 1)
+    (in_bom yes) (on_board yes) (fields_autoplaced)
+    (property "Reference" "IC1" (id 0) (at 457.2 228.5999 0)
+      (effects (font (size 1.27 1.27)) (justify left))
+    )
+    (property "Value" "4A 8D1" (id 1) (at 457.2 231.1399 0)
+      (effects (font (size 1.27 1.27)) (justify left))
+    )
+    (property "Footprint" "Gameboy Printer:SOT89 Transistor" (id 2) (at 457.2 227.33 0)
+      (effects (font (size 1.27 1.27)) hide)
+    )
+    (property "Datasheet" "~" (id 3) (at 462.28 229.87 0)
+      (effects (font (size 1.27 1.27)) hide)
+    )
+    (pin "1")
+    (pin "2")
+    (pin "3")
   )
   (symbol (lib_id "Device:Q_NPN_BEC") (at 374.65 265.43 90) (mirror x) (unit 1)
@@
     (pin "2")
   )
-  (symbol (lib_id "Amplifier_Operational:TL064") (at 459.74 229.87 0) (mirror x) (unit 1)
-    (in_bom yes) (on_board yes)
-    (property "Reference" "IC1" (id 0) (at 455.93 241.3 0))
-    (property "Value" "4A 8D1 - BGA6489" (id 1) (at 455.93 238.76 0))
-    (property "Footprint" "Gameboy Printer:SOT89 Transistor" (id 2) (at 458.47 232.41 0)
-      (effects (font (size 1.27 1.27)) hide)
-    )
-    (property "Datasheet" "http://www.ti.com/lit/ds/symlink/tl061.pdf" (id 3) (at 461.01 234.95 0)
-      (effects (font (size 1.27 1.27)) hide)
-    )
-    (pin "1")
-    (pin "2")
-    (pin "3")
-  )
   (symbol (lib_id "Device:R_Small_US") (at 396.24 182.88 180) (unit 1)
     (in_bom yes) (on_board yes)
@@
       (reference "F2") (unit 1) (value "102C Thermal Fuse") (footprint "Gameboy Printer:F2 Thermal Fuse")
     )
-    (path "/9d05feb3-8bdf-4b65-8875-c4c57a254f42"
-      (reference "IC1") (unit 1) (value "4A 8D1 - BGA6489") (footprint "Gameboy Printer:SOT89 Transistor")
+    (path "/0c144793-bba0-4892-9883-fd3891cc63cb"
+      (reference "IC1") (unit 1) (value "4A 8D1") (footprint "Gameboy Printer:SOT89 Transistor")
     )
     (path "/62b9d962-6a37-4ac5-bd9c-e9c0b700b0ec"

Commit message: Add files via upload
Connections:
- net GND: no longer C1.1, F2.1, Q1.3 (E), R1.1, R16.2, R17.2, R21.1
- new net: C1.1, F2.1, Q1.3 (E), R1.1, R16.2, R17.2, R21.1
Changed lines of the file:
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@@
-    (stroke (width 0) (type default) (color 0 0 0 0))
-  )
-  (wire (pts (xy 477.52 325.12) (xy 477.52 320.04))
     (stroke (width 0) (type default) (color 0 0 0 0))
   )
